File: pcb_design/reference pcb_cad/Adafruit-Pro-Trinket-PCBs-master/Adafruit Pro Trinket 3v3.sch (EAGLE design)
At the start: 26 parts, among them IC1 ATmega328P, IC2 MIC5225-3.3v, Q1 reset, Y1 12MHz

Commit message: added a bunch of new stuff in
Other:
- moved on the sheet: CN1
Changed lines of the file:
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@@
 <?xml version="1.0" encoding="utf-8"?>
 <!DOCTYPE eagle SYSTEM "eagle.dtd">
-<eagle version="6.3">
+<eagle version="7.5.0">
 <drawing>
 <settings>
@@
 <instance part="B1" gate="G$1" x="134.62" y="109.22" rot="MR180"/>
 <instance part="GND4" gate="1" x="139.7" y="106.68"/>
-<instance part="CN1" gate="G$1" x="121.92" y="134.62"/>
+<instance part="CN1" gate="G$1" x="119.38" y="134.62"/>
 <instance part="U$2" gate="G$1" x="134.62" y="142.24"/>
 <instance part="IC1" gate="G$1" x="63.5" y="142.24"/>
@@
 <net name="GND" class="1">
 <segment>
-<wire x1="132.08" y1="129.54" x2="139.7" y2="129.54" width="0.1524" layer="91"/>
+<wire x1="129.54" y1="129.54" x2="139.7" y2="129.54" width="0.1524" layer="91"/>
 <wire x1="139.7" y1="129.54" x2="139.7" y2="127" width="0.1524" layer="91"/>
 <pinref part="GND1" gate="1" pin="GND"/>
@@
 <net name="D+" class="0">
 <segment>
-<wire x1="132.08" y1="137.16" x2="137.16" y2="137.16" width="0.1524" layer="91"/>
+<wire x1="129.54" y1="137.16" x2="137.16" y2="137.16" width="0.1524" layer="91"/>
 <wire x1="137.16" y1="137.16" x2="142.24" y2="132.08" width="0.1524" layer="91"/>
 <wire x1="142.24" y1="132.08" x2="149.86" y2="132.08" width="0.1524" layer="91"/>
@@
 <net name="D-" class="0">
 <segment>
-<wire x1="132.08" y1="134.62" x2="137.16" y2="134.62" width="0.1524" layer="91"/>
+<wire x1="129.54" y1="134.62" x2="137.16" y2="134.62" width="0.1524" layer="91"/>
 <wire x1="137.16" y1="134.62" x2="139.7" y2="137.16" width="0.1524" layer="91"/>
 <pinref part="R1" gate="G$1" pin="1"/>
@@
 <pinref part="CN1" gate="G$1" pin="VBUS"/>
 <pinref part="U$2" gate="G$1" pin="VBUS"/>
-<wire x1="134.62" y1="139.7" x2="132.08" y2="139.7" width="0.1524" layer="91"/>
-</segment>
-<segment>
+<wire x1="134.62" y1="139.7" x2="129.54" y2="139.7" width="0.1524" layer="91"/>
+</segment>
+<segment>
