File: pcb_design/reference pcb_cad/Adafruit-Pro-Trinket-PCBs-master/Adafruit Pro Trinket 5v0.sch (EAGLE design)
At the start: 28 parts, among them CN2 JSTPH, IC1 ATmega328P, Q1 reset, U1 MCP73831T-2ACI/OT, Y1 16MHz

Commit message: added a bunch of new stuff in
Parts:
- removed B2: red, microbuilder:LED0805_NOOUTLINE
- removed C4: 10µF, microbuilder:CAP_CERAMIC0805-NOOUTLINE
- removed CN2: JSTPH, microbuilder:JST_2PIN
- removed JP3: (no value), SparkFun:M03JST-PTH
- removed LED2: GREEN, microbuilder:LED0805_NOOUTLINE
- removed R8: 470, microbuilder:RESISTOR0805_NOOUTLINE
- removed R9: 10K\, microbuilder:RESISTOR0805_NOOUTLINE
- removed U1: MCP73831T-2ACI/OT, microbuilder:MCP73831/2
- added BAT: JST 2-PH, microbuilder:CON_JST_PH_2PIN
- added C8: 10uF, microbuilder:CAP_CERAMIC0805-NOOUTLINE
- added D2: SCHOTTKY, adafruit:DIODE_SOD-123FL
- added IC2: MIC5225-5v, adafruit:LP298XS
- added JP2: (no value), microbuilder:HEADER-1X2ROUND
- added JP4: (no value), adafruit:PINHD-1X12-CB
- added PWR: green, microbuilder:LED0805_NOOUTLINE
- C1: value 10µF -> 10uF
- JP1: device microbuilder:HEADER-1X2ROUND -> adafruit:PINHD-1X12-CB
Connections:
- removed net N$4: B2.A, R4.1
- removed net N$7: R9.1, U1.PROG
- removed net N$8: LED2.A, R8.1
- removed net STRIP_CNTRL: JP3.2
- removed net VBAT1: C4.1, CN2.2, JP1.2, U1.VBAT
- new net VBAT: BAT.2, C1.1, IC2.EN, IC2.VIN, JP1.1
- net +5V: now also C8.1, D2.C, IC2.VOUT, JP1.4; no longer C1.1, CN1.VBUS, JP1.1, JP3.3, U1.VDD
- net A0: now also JP4.7
- net A1: now also JP4.8
- net A2: now also JP4.9
- net A3: now also JP4.10
- net A4: now also JP4.11
- net A5: now also JP4.12
- net A6: now also JP2.1
- net A7: now also JP2.2
- net AREF: now also JP4.6
- net D10: now also JP4.2
- net D11: now also JP4.3
- net D12: now also JP4.4
- net D13: now also JP4.5
- net D3: now also JP1.9
- net D4: now also JP1.8
- net D5: now also JP1.7
- net D6: now also JP1.6
- net D8: now also JP1.5
- net D9: now also JP4.1
- net GND: now also BAT.1, C8.2, IC2.GND, JP1.2, PWR.C; no longer B2.C, C4.2, CN2.1, JP3.1, LED2.C, R9.2, U1.VSS
- net N$6: now also PWR.A, R4.1; no longer R8.2, U1.STAT
- net RESET: now also JP1.12
- net RXD: now also JP1.11
- net TXD: now also JP1.10
- net VBUS: now also CN1.VBUS, D2.A, JP1.3
Other:
- note removed: "1.0K = 1000mA"
- note removed: "10K = 100mA"
- note removed: "2.0K = 500mA"
- note removed: "5.0K = 200mA"
- note removed: "Assembly and use note : If you plan to do USB-powered operation, do not populate the Battery Charge electronics. Instead you need to solder JP1 shut"
- note removed: "Battery Charger Circuit"
- note removed: "USB Data and Power In"
- note removed: "USB power LED"
- moved on the sheet: B1, C1, CN1, D1, D4, R1, R2, R3, R4, R5
