File: pcb_design/Light_node.brd (EAGLE design)
At the start: 26.8 x 37.3 mm, 38 parts, among them CN3 JSTPH, IC1 ATmega328P, IC2 MIC5225-3.3v, U1 MCP73831T-2ACI/OT, U2 LIS3DHTR, Y1 12MHz

Commit message: Things are pretty close to complete
Parts:
- removed C1, C8: 10uF, microbuilder:0805-NO
- removed C2: 0.1uF, microbuilder:_0805MP
- removed C3: 0.1uF, microbuilder:0805-NO
- removed C4, C5, C7: 10µF, microbuilder:0805-NO
- removed CN1: (no value), microbuilder:4UCONN_20329
- removed CN3: JSTPH, microbuilder:JSTPH2
- removed D3: SCHOTTKY, adafruit:SOD-123FL
- removed IC1: ATmega328P, microbuilder:MLF32-TH
- removed IC2: MIC5225-3.3v, adafruit:SOT23-5L
- removed LED3, LED4: WS2812B5050, microbuilder:WS2812B
- removed R12: 10K\, microbuilder:0805-NO
- removed R16, R8: 10K, microbuilder:0805-NO
- removed R4: 470 (0603), microbuilder:0603-NO
- removed R6: 10K (0603), microbuilder:0805-NO
- removed R7: TRIMPOT, SparkFun:3362U-2
- removed U$9: COMMON_ANODE_DIODE, 0_AlpineLabs:SOT23
- removed U1: MCP73831T-2ACI/OT, microbuilder:SOT23-5
- removed U2: LIS3DHTR, microbuilder:LGA16_3X3MM
- removed Y1: 12MHz, SparkFun:RESONATOR-SMD
- added C10, C11, C20: 10µF, microbuilder:0805-NO
- added C30: 0.1uF, microbuilder:_0805MP
- added C31: 0.1uF, microbuilder:0805-NO
- added C40, C41: 10uF, microbuilder:0805-NO
- added D40: SCHOTTKY, adafruit:SOD-123FL
- added JP11: (no value), microbuilder:1X02_ROUND
- added JP3: JSTPH, microbuilder:JSTPH2
- added POT: (no value), 0_Shibbs1:3306P_POT
- added R20, R21: 10K, microbuilder:0805-NO
- added R30: 10K (0603), microbuilder:0805-NO
- added R40: 470 (0603), microbuilder:0603-NO
- added R50: 10K, microbuilder:0603-NO
- added RGB1, RGB2: WS2812B5050, microbuilder:WS2812B
- added U10: MCP73831T-2ACI/OT, microbuilder:SOT23-5
- added U20: LIS3DHTR, microbuilder:LGA16_3X3MM
- added U30: ATmega328P, microbuilder:MLF32-TH
- added U40: MIC5225-3.3v, adafruit:SOT23-5L
- added U50: COMMON_ANODE_DIODE, 0_AlpineLabs:SOT23
- added Y30: 12MHz, SparkFun:RESONATOR-SMD
- JP1: value (none) -> USB_MICROB_PLUG_CUSTOM; device SparkFun:JST-3-PTH -> 0_AlpineLabs:USB-MICROB
- JP5: value (none) -> M03; device microbuilder:1X02_ROUND -> 0_Shibbs1:M03_25MM
- R10: value 10K -> 470; device microbuilder:0603-NO -> microbuilder:0805-NO
- R11: value 470 -> 10K\
- moved JP1 28.8 mm to (6.80, 34.2), turned to 180 degrees
- moved JP5 16.0 mm to (21.2, 12.5), turned to 0 degrees
- moved R10 15.8 mm to (20.1, 32.0)
- moved R11 7.33 mm to (22.1, 26.6), turned to 90 degrees
- moved R2 4.29 mm to (4.87, 26.3)
- moved R5 4.29 mm to (3.24, 26.3)
- moved R1 4.11 mm to (6.47, 26.3)
- moved R3 3.93 mm to (8.06, 26.3)
- moved R9 3.93 mm to (14.3, 19.4)
- moved B1 3.93 mm to (3.01, 29.2)
- moved CH_LED 3.93 mm to (16.4, 34.3)
- moved FTDI 3.93 mm to (8.49, 1.49)
- moved JP2 3.93 mm to (24.5, 16.2)
- moved PWR_LED 3.93 mm to (10.6, 29.2)
Connections:
- removed net 3.3V: C7.1, R8.2, U2.1, U2.14
- removed net INT1: U2.11
- net +3V3: now also C20.1, C41.1, JP2.10, POT.P$1, R20.2, R30.2, R40.2, U20.1, U20.14, U30.18, U30.4, U30.6, U40.5, U50.1; no longer C8.1, IC1.18, IC1.4, IC1.6, IC2.5, R4.2, R6.2, R7.3, U$9.1
- net +5V: now also C10.1, C40.1, D40.C, JP1.VBUS, JP11.1, JP2.11, JP5.P$3, R50.1, U10.4, U40.1, U40.3; no longer C1.1, C4.1, CN1.VBUS, D3.C, IC2.1, IC2.3, JP1.1, JP5.1, R10.1, U1.4
- net A0: now also U30.23; no longer IC1.23
- net A1: now also JP2.2, U30.24; no longer IC1.24
- net A2: now also JP2.1, U20.11, U30.25; no longer IC1.25
- net A3: now also U30.26; no longer IC1.26
- net A6: now also JP2.3, U30.19; no longer IC1.19
- net A7: now also POT.P$3, U30.22; no longer IC1.22, R7.2
- net ADC1: now also U20.16; no longer U2.16
- net ADC2: now also U20.15; no longer U2.15
- net ADC3: now also U20.13; no longer U2.13
- net AREF: now also C30.1, U30.20; no longer C2.1, IC1.20
- net CS: now also R20.1, U20.8; no longer R8.1, U2.8
- net D+: now also JP1.D+; no longer CN1.D+
- net D-: now also JP1.D-; no longer CN1.D-
- net D10: now also U30.14; no longer IC1.14
- net D11: now also JP2.7, U30.15; no longer IC1.15
- net D12: now also JP2.8, U30.16; no longer IC1.16
- net D13: now also U30.17; no longer IC1.17
- net D2: now also U30.32; no longer IC1.32
- net D3: now also JP2.4, U30.1; no longer IC1.1
- net D4: now also U30.2, U50.2; no longer IC1.2, U$9.2
- net D5: now also JP2.5, U30.9; no longer IC1.9
- net D6: now also JP2.6, U30.10; no longer IC1.10
- net D7: now also U30.11; no longer IC1.11
- net D8: now also U30.12; no longer IC1.12
- net D9: now also U30.13; no longer IC1.13
- net DTR/RTS: now also C31.2; no longer C3.2
- net GND: now also C10.2, C11.2, C20.2, C30.2, C40.2, C41.2, JP1.GND, JP1.P$1, JP1.P$2, JP1.P$3, JP1.P$4, JP2.12, JP3.1, JP5.P$2, POT.P$2, R11.2, R21.1, RGB1.3-GND, RGB2.3-GND, U10.2, U20.10, U20.12, U20.5, U30.21, U30.3, U30.5, U30.TH, U40.2, Y30.2; no longer C1.2, C2.2, C4.2, C5.2, C7.2, C8.2, CN1.BASE@1, CN1.BASE@2, CN1.GND, CN1.SPRT@1, CN1.SPRT@2, CN1.SPRT@3, CN1.SPRT@4, CN3.1, IC1.21, IC1.3, IC1.5, IC1.TH, IC2.2, JP1.2, LED3.3-GND, LED4.3-GND, R12.2, R16.1, R7.1, U1.2, U2.10, U2.12, U2.5, Y1.2
- net LED_CNTRL: now also RGB1.4-DIN; no longer LED3.4-DIN
- net N$15: now also RGB2.2-DOUT; no longer LED4.2-DOUT
- net N$2: now also U30.8, Y30.3; no longer IC1.8, Y1.3
- net N$3: now also U30.7, Y30.1; no longer IC1.7, Y1.1
- net N$4: now also RGB1.2-DOUT, RGB2.4-DIN; no longer LED3.2-DOUT, LED4.4-DIN
- net N$5: now also R10.2, U10.1; no longer R11.2, U1.1
- net N$6: now also R40.1; no longer R4.1
- net N$8: now also R11.1, U10.5; no longer R12.1, U1.5
- net N$9: now also R10.1; no longer R11.1
- net RESET: now also C31.1, R30.1, U30.29; no longer C3.1, IC1.29, R6.1
- net RXD: now also U30.30; no longer IC1.30
- net SCL: now also U20.4, U30.28; no longer IC1.28, U2.4
- net SDA: now also U20.6, U30.27; no longer IC1.27, U2.6
- net SDO: now also R21.2, U20.7; no longer R16.2, U2.7
- net STRIP_CNTRL: now also JP5.P$1, R50.2, U50.3; no longer JP1.3, R10.2, U$9.3
- net TXD: now also U30.31; no longer IC1.31
- net VBAT: now also C11.1, D40.A, JP11.2, JP2.9, JP3.2, RGB1.1-VDD, RGB2.1-VDD, U10.3; no longer C5.1, CN3.2, D3.A, JP5.2, LED3.1-VDD, LED4.1-VDD, U1.3
Routing:
- net A2: track 0.16 -> 42.2 mm, vias 0 -> 2
- net GND: track 65.3 -> 107.3 mm, vias 7 -> 19
- net +3V3: track 44.7 -> 82.6 mm, vias 4 -> 5
- net A6: track 1.07 -> 27.2 mm, vias 0 -> 2
- net A1: track 0.00 -> 24.5 mm, vias 0 -> 1
- net +5V: track 72.9 -> 88.7 mm, vias 3 -> 6
- net D12: track 10.2 -> 21.8 mm
- net D5: track 6.27 -> 17.7 mm
- net D11: track 9.83 -> 20.5 mm
- net D6: track 6.46 -> 16.3 mm
- net 3.3V: track 8.20 -> 0.00 mm
- net D3: track 8.11 -> 15.8 mm
- net VBAT: track 53.6 -> 60.4 mm
- net STRIP_CNTRL: track 4.71 -> 8.75 mm
- net N$4: track 15.9 -> 18.4 mm
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Other:
- board outline removed
- board text added: "Charging"
- board text added: "Gnd"
- board text added: "Light Node V1"
- board text removed: "12 MHz"
- board text removed: "3V"
- board text removed: "5V"
- board text removed: "A5"
- board text removed: "BLK"
- board text removed: "FTDI Header"
- board text removed: "GND"
- board text removed: "GRN"
- board text removed: "Pro"
- board text removed: "RST"
- board text removed: "RX"
- board text removed: "TX"
- board text removed: "Trinket!"
