File: pcb_design/Light_node.brd (EAGLE design)
At the start: 39 parts, among them U10 MCP73831T-2ACI/OT, U20 LIS3DHTR, U30 ATmega328P, U40 MIC5225-3.3v, U50 COMMON_ANODE_DIODE, Y30 12MHz

Commit message: got the boards running and initial code is working well!!!
Parts:
- R9: value 100 -> 470; device microbuilder:0603-NO -> 0_shibbs2:0603-RES
Changed lines of the file:
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@@
 <attribute name="NAME" x="15.2556" y="16.3666" size="1.27" layer="25" font="vector" ratio="18"/>
 </element>
-<element name="R9" library="microbuilder" package="0603-NO" value="100" x="14.2936" y="19.4224" smashed="yes" rot="R180">
+<element name="R9" library="0_shibbs2" package="0603-RES" value="470" x="14.2936" y="19.4224" smashed="yes" rot="R180">
 <attribute name="NAME" x="15.5156" y="21.5494" size="1.27" layer="25" font="vector" ratio="18" rot="R180"/>
 </element>
